File: KiCad/Lab4/exercise 1/Lab4.kicad_sch (KiCad schematic)
At the start: 6 parts, among them SW1 SW_SPDT

Commit message: updated lab4
Parts:
- C1: footprint (none) -> Capacitor_THT:C_Radial_D5.0mm_H5.0mm_P2.00mm
- D1: footprint (none) -> LED_THT:LED_D5.0mm
- R1, R2: footprint (none) -> Resistor_THT:R_Axial_DIN0516_L15.5mm_D5.0mm_P20.32mm_Horizontal
- SW1: footprint (none) -> Button_Switch_THT:SW_E-Switch_EG1224_SPDT_Angled
- V1: footprint (none) -> Connector_JST:JST_PH_B2B-PH-K_1x02_P2.00mm_Vertical
Connections:
- net at SW1.2 (B): now also R2.2
Other:
- moved on the sheet: SW1
Changed lines of the file:
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@@
   (junction (at 116.84 64.77) (diameter 0) (color 0 0 0 0)
   )
-  (wire (pts (xy 107.95 64.77) (xy 116.84 64.77))
+  (wire (pts (xy 110.49 64.77) (xy 116.84 64.77))
     (stroke (width 0) (type default) (color 0 0 0 0))
   )
@@
     (stroke (width 0) (type default) (color 0 0 0 0))
   )
-  (wire (pts (xy 87.63 62.23) (xy 101.6 62.23))
+  (wire (pts (xy 142.24 64.77) (xy 142.24 66.04))
     (stroke (width 0) (type default) (color 0 0 0 0))
   )
-  (wire (pts (xy 142.24 64.77) (xy 142.24 66.04))
+  (wire (pts (xy 87.63 62.23) (xy 100.33 62.23))
     (stroke (width 0) (type default) (color 0 0 0 0))
   )
@@
       (effects (font (size 1.27 1.27)) (justify right))
     )
-    (property "Footprint" "" (id 2) (at 142.24 90.17 0)
+    (property "Footprint" "LED_THT:LED_D5.0mm" (id 2) (at 142.24 90.17 0)
       (effects (font (size 1.27 1.27)) hide)
     )
@@
     (pin "2")
   )
-  (symbol (lib_id "Switch:SW_SPDT") (at 102.87 62.23 0) (unit 1)
+  (symbol (lib_id "Switch:SW_SPDT") (at 105.41 62.23 0) (unit 1)
     (in_bom yes) (on_board yes) (fields_autoplaced)
-    (property "Reference" "SW1" (id 0) (at 102.87 54.61 0))
-    (property "Value" "SW_SPDT" (id 1) (at 102.87 57.15 0))
-    (property "Footprint" "" (id 2) (at 102.87 62.23 0)
+    (property "Reference" "SW1" (id 0) (at 105.41 54.61 0))
+    (property "Value" "SW_SPDT" (id 1) (at 105.41 57.15 0))
+    (property "Footprint" "Button_Switch_THT:SW_E-Switch_EG1224_SPDT_Angled" (id 2) (at 105.41 62.23 0)
       (effects (font (size 1.27 1.27)) hide)
     )
-    (property "Datasheet" "~" (id 3) (at 102.87 62.23 0)
+    (property "Datasheet" "~" (id 3) (at 105.41 62.23 0)
       (effects (font (size 1.27 1.27)) hide)
     )
@@
       (effects (font (size 1.27 1.27)) (justify right))
     )
-    (property "Footprint" "" (id 2) (at 115.8748 72.39 0)
+    (property "Footprint" "Capacitor_THT:C_Radial_D5.0mm_H5.0mm_P2.00mm" (id 2) (at 115.8748 72.39 0)
       (effects (font (size 1.27 1.27)) hide)
     )
@@
       (effects (font (size 1.27 1.27)) (justify left))
     )
-    (property "Footprint" "" (id 2) (at 140.462 69.85 90)
+    (property "Footprint" "Resistor_THT:R_Axial_DIN0516_L15.5mm_D5.0mm_P20.32mm_Horizontal" (id 2) (at 140.462 69.85 90)
       (effects (font (size 1.27 1.27)) hide)
     )
@@
     (property "Reference" "R2" (id 0) (at 83.82 55.88 90))
     (property "Value" "2.2K" (id 1) (at 83.82 58.42 90))
-    (property "Footprint" "" (id 2) (at 83.82 64.008 90)
+    (property "Footprint" "Resistor_THT:R_Axial_DIN0516_L15.5mm_D5.0mm_P20.32mm_Horizontal" (id 2) (at 83.82 64.008 90)
       (effects (font (size 1.27 1.27)) hide)
     )
@@
     (property "Reference" "V1" (id 0) (at 67.945 71.12 0))
     (property "Value" "9 V" (id 1) (at 67.945 73.66 0))
-    (property "Footprint" "" (id 2) (at 67.31 76.2 0)
+    (property "Footprint" "Connector_JST:JST_PH_B2B-PH-K_1x02_P2.00mm_Vertical" (id 2) (at 67.31 76.2 0)
       (effects (font (size 1.27 1.27)) hide)
     )
@@
   (symbol_instances
     (path "/87e84922-8127-4fd7-9cb2-ed8e95402210"
-      (reference "C1") (unit 1) (value "4.7 uF") (footprint "")
+      (reference "C1") (unit 1) (value "4.7 uF") (footprint "Capacitor_THT:C_Radial_D5.0mm_H5.0mm_P2.00mm")
     )
     (path "/486d635e-ff0b-40ea-820d-b78722e331e8"
-      (reference "D1") (unit 1) (value "LED") (footprint "")
+      (reference "D1") (unit 1) (value "LED") (footprint "LED_THT:LED_D5.0mm")
     )
     (path "/a751aff6-00fc-4a98-9431-edecd4830404"
-      (reference "R1") (unit 1) (value "20K") (footprint "")
+      (reference "R1") (unit 1) (value "20K") (footprint "Resistor_THT:R_Axial_DIN0516_L15.5mm_D5.0mm_P20.32mm_Horizontal")
     )
     (path "/d941e45a-f215-4b1c-8803-a70eb09b3edf"
-      (reference "R2") (unit 1) (value "2.2K") (footprint "")
+      (reference "R2") (unit 1) (value "2.2K") (footprint "Resistor_THT:R_Axial_DIN0516_L15.5mm_D5.0mm_P20.32mm_Horizontal")
     )
     (path "/76689453-c418-4de0-a02e-d6bbb08d342a"
-      (reference "SW1") (unit 1) (value "SW_SPDT") (footprint "")
+      (reference "SW1") (unit 1) (value "SW_SPDT") (footprint "Button_Switch_THT:SW_E-Switch_EG1224_SPDT_Angled")
     )
     (path "/f3d3f191-849a-417e-b2fd-dd3d4ba80f77"
-      (reference "V1") (unit 1) (value "9 V") (footprint "")
+      (reference "V1") (unit 1) (value "9 V") (footprint "Connector_JST:JST_PH_B2B-PH-K_1x02_P2.00mm_Vertical")
     )
   )
